File: IOT/kicad/wifi.kicad_sch (KiCad schematic)
At the start: 2 parts

Commit message: docs(iot): kicad pbl0 pbl1
Connections:
- no-connect marks 2 -> 4
Changed lines of the file:
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@@
+	)
+	(no_connect
+		(at 48.26 49.53)
 	)
 	(no_connect
@@
 	)
 	(no_connect
+		(at 48.26 54.61)
+	)
+	(no_connect
