File: IOT/kicad/poubelle3.kicad_sch (KiCad schematic)
At the start: 0 parts

Commit message: docs: fix bins' names in kicad
Other:
- title: Poubelle 3 -> Poubelle 2
Changed lines of the file:
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@@
 	(paper "A5")
 	(title_block
-		(title "Poubelle 3")
+		(title "Poubelle 2")
 		(rev "0.0.1")
 	)

Commit message: docs(iot): pbl 1 & 2
Parts:
- added LCD-1: ~, symbol OrdureX:LCD-1602
- added MatrixMembraneKeypad1: ~, symbol OrdureX:27899
- added R2, R3: R, symbol Device:R
- added R4: 10k, symbol Device:R
- added SG1: Motor Servo (SrvM), symbol Motor:Motor_Servo
Connections:
- net GND: now also LCD-1.1 (VSS), LCD-1.5 (RW), R3.2, SG1.3 (-)
- new net: LCD-1.16 (K), R3.1
- new net: R4.1, SG1.2 (+)
- new net: LCD-1.3 (VO), R2.1
- new net 5V: LCD-1.15 (A), LCD-1.2 (VDD), R2.2, R4.2
- new net Keypad-1: MatrixMembraneKeypad1.0 (D0)
- new net Keypad-2: MatrixMembraneKeypad1.1 (D1)
- new net Keypad-3: MatrixMembraneKeypad1.2 (D2)
- new net Keypad-4: MatrixMembraneKeypad1.3 (D3)
- new net Keypad-5: MatrixMembraneKeypad1.4 (D4)
- new net Keypad-6: MatrixMembraneKeypad1.5 (D5)
- new net Keypad-7: MatrixMembraneKeypad1.6 (D6)
- new net LCD-D4: LCD-1.11 (D4)
- new net LCD-D5: LCD-1.12 (D5)
- new net LCD-D6: LCD-1.13 (D6)
- new net LCD-D7: LCD-1.14 (D7)
- new net LCD-E: LCD-1.6 (E)
- new net LCD-RS: LCD-1.4 (RS)
- new net SrvM2-PWM-IN: SG1.1 (PWM)
- no-connect marks 0 -> 5
