File: IOT/kicad/ordurex-electronics.kicad_sch (KiCad schematic)
At the start: 1 part

Commit message: docs(kicad): fix pin of servomotors
Connections:
- net Poubelle 0/SrvM1-PWM-IN: now also A1.D23; no longer A1.D4
- net Poubelle 2/SrvM2-PWM-IN: now also A1.D24; no longer A1.D10
Changed lines of the file:
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@@
+	(wire
+		(pts
+			(xy 166.37 59.69) (xy 190.5 59.69)
+		)
+		(stroke
+			(width 0)
+			(type default)
+		)
+	)
 	(wire
 		(pts
@@
 	(wire
 		(pts
+			(xy 204.47 59.69) (xy 204.47 62.23)
+		)
+		(stroke
+			(width 0)
+			(type default)
+		)
+	)
+	(wire
+		(pts
 			(xy 187.96 39.37) (xy 208.28 39.37)
 		)
@@
 	(wire
 		(pts
-			(xy 195.58 59.69) (xy 195.58 46.99)
-		)
-		(stroke
-			(width 0)
-			(type default)
-		)
-	)
-	(wire
-		(pts
 			(xy 236.22 35.56) (xy 240.03 35.56)
 		)
@@
 	(wire
 		(pts
+			(xy 190.5 43.18) (xy 190.5 59.69)
+		)
+		(stroke
+			(width 0)
+			(type default)
+		)
+	)
+	(wire
+		(pts
 			(xy 166.37 90.17) (xy 208.28 90.17)
 		)
@@
 	(wire
 		(pts
-			(xy 166.37 31.75) (xy 208.28 31.75)
-		)
-		(stroke
-			(width 0)
-			(type default)
-		)
-	)
-	(wire
-		(pts
-			(xy 208.28 59.69) (xy 195.58 59.69)
+			(xy 208.28 59.69) (xy 204.47 59.69)
 		)
 		(stroke
@@
 	(wire
 		(pts
+			(xy 166.37 62.23) (xy 204.47 62.23)
+		)
+		(stroke
+			(width 0)
+			(type default)
+		)
+	)
+	(wire
+		(pts
 			(xy 240.03 129.54) (xy 240.03 132.08)
 		)
@@
 	(wire
 		(pts
+			(xy 190.5 43.18) (xy 208.28 43.18)
+		)
+		(stroke
+			(width 0)
+			(type default)
+		)
+	)
+	(wire
+		(pts
 			(xy 240.03 63.5) (xy 240.03 66.04)
 		)
@@
 			(type default)
 			(color 255 0 0 1)
-		)
-	)
-	(wire
-		(pts
-			(xy 195.58 46.99) (xy 166.37 46.99)
-		)
-		(stroke
-			(width 0)
-			(type default)
 		)
 	)
@@
 		)
 		(pin "SrvM1-PWM-IN" input
-			(at 208.28 31.75 180)
-			(effects
-				(font
+			(at 208.28 43.18 180)
+			(effects
+				(font
