File: IOT/kicad/poubelle1.kicad_sch (KiCad schematic)
At the start: 3 parts, among them M1 Motor_Servo

Commit message: docs: fix bins' names in kicad
Other:
- title: Poubelle 1 -> Poubelle 0
Changed lines of the file:
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@@
 	(paper "A5")
 	(title_block
-		(title "Poubelle 1")
+		(title "Poubelle 0")
 		(date "2024-05-21")
 		(rev "0.0.1")

Commit message: docs(iot): kicad pbl0 pbl1
Parts:
- KY-032: renamed from HC-SR1; value ~ -> Infrared obstacle sensor
- SG90: renamed from M1; value Motor_Servo -> Motor Servo (SrvM)
Connections:
- net 5V_PS renamed 5V
- net 5V: no longer KY-032.0 (VCC)
- net D1 renamed SrvM-PWM-IN
- net GND_ARD: no longer names the net of KY-032.3 (EN)
- net GND_ARD: no longer SG90.3 (-)
- net RX renamed KY32-out
- net TX renamed 3.3V
- new net GND: KY-032.0 (GND), SG90.3 (-)
- no-connect marks 0 -> 1
Other:
- note removed: "ARD: Arduino PS: Power supply (non arduino)"
- moved on the sheet: KY-032, R1

Commit message: docs(iot): pbl 1 & 2
Connections:
- net SrvM-PWM-IN renamed SrvM1-PWM-IN
Changed lines of the file:
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@@
 		)
 	)
-	(hierarchical_label "SrvM-PWM-IN"
+	(hierarchical_label "SrvM1-PWM-IN"
 		(shape input)
 		(at 111.76 62.23 0)

Commit message: docs(iot): kicad filename + resistance + typo
Parts:
- removed KY-032: Infrared obstacle sensor, symbol OrdureX:HC-SR04
- removed R1: 10k, symbol Device:R
- removed SG90: Motor Servo (SrvM), symbol Motor:Motor_Servo
- added KY-006: buzzer, symbol OrdureX:KY-006
- added KY-026: fire sensor, symbol OrdureX:KY-026
- added RFID-RC1: ~, symbol OrdureX:RFID-RC522
Connections:
- net 3.3V: now also KY-026.2 (3.3-5V), RFID-RC1.7 (VCC)
- net GND: now also KY-006.2 (GND), KY-026.1 (GND), RFID-RC1.5 (GND)
- new net KY26-out: KY-026.0 (D0)
- new net KY6-in: KY-006.0 (D0)
- new net RFID-MISO: RFID-RC1.3 (MISO)
- new net RFID-MOSI: RFID-RC1.2 (MOSI)
- new net RFID-RST: RFID-RC1.6 (RST)
- new net RFID-SCLK: RFID-RC1.1 (SCLK)
- new net RFID-SDA: RFID-RC1.0 (SDA)
- no-connect marks 1 -> 3
Other:
- title: Poubelle 0 -> Poubelle 1
