File: IOT/kicad/poubelle2.kicad_sch (KiCad schematic)
At the start: 1 part

Commit message: docs: fix bins' names in kicad
Other:
- title: Poubelle 2 -> Poubelle 1
Changed lines of the file:
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@@
 	(paper "A5")
 	(title_block
-		(title "Poubelle 2")
+		(title "Poubelle 1")
 		(rev "0.0.1")
 	)

Commit message: docs(iot): kicad pbl0 pbl1
Parts:
- added KY-006: buzzer, symbol OrdureX:KY-006
- added KY-026: fire sensor, symbol OrdureX:KY-026
Connections:
- net D0 renamed Keypad-1
- net D1 renamed Keypad-2
- net D2 renamed Keypad-3
- net D3 renamed Keypad-4
- net D4 renamed Keypad-5
- net D5 renamed Keypad-6
- net D6 renamed Keypad-7
- net D7 renamed Keypad-8
- new net 3.3V: KY-026.2 (3.3-5V)
- new net GND: KY-006.2 (GND), KY-026.1 (GND)
- new net K6-in: KY-006.0 (D0)
- new net KY26-out: KY-026.0 (D0)
- no-connect marks 0 -> 2
Other:
- moved on the sheet: MatrixMembraneKeypad

Commit message: docs(iot): pbl 1 & 2
Parts:
- removed MatrixMembraneKeypad: ~, symbol OrdureX:27899
- added RFID-RC1: ~, symbol OrdureX:RFID-RC522
Connections:
- net 3.3V: now also RFID-RC1.7 (VCC)
- net GND: now also RFID-RC1.5 (GND)
- new net RFID-MISO: RFID-RC1.3 (MISO)
- new net RFID-MOSI: RFID-RC1.2 (MOSI)
- new net RFID-RST: RFID-RC1.6 (RST)
- new net RFID-SCLK: RFID-RC1.1 (SCLK)
- new net RFID-SDA: RFID-RC1.0 (SDA)
- no-connect marks 2 -> 3
Other:
- moved on the sheet: KY-006, KY-026

Commit message: docs(iot): kicad filename + resistance + typo
Parts:
- removed KY-006: buzzer, symbol OrdureX:KY-006
- removed KY-026: fire sensor, symbol OrdureX:KY-026
- removed RFID-RC1: ~, symbol OrdureX:RFID-RC522
- added LCD-1: ~, symbol OrdureX:LCD-1602
- added MatrixMembraneKeypad1: ~, symbol OrdureX:27899
- added R2: 330, symbol Device:R
- added R3: 1k, symbol Device:R
- added R4: 10k, symbol Device:R
- added SG1: Motor Servo (SrvM), symbol Motor:Motor_Servo
Connections:
- net GND: now also LCD-1.1 (VSS), LCD-1.5 (RW), R3.2, SG1.3 (-)
- new net: LCD-1.16 (K), R3.1
- new net: R4.1, SG1.2 (+)
- new net: LCD-1.3 (VO), R2.1
- new net 5V: LCD-1.15 (A), LCD-1.2 (VDD), R2.2, R4.2
- new net Keypad-1: MatrixMembraneKeypad1.0 (D0)
- new net Keypad-2: MatrixMembraneKeypad1.1 (D1)
- new net Keypad-3: MatrixMembraneKeypad1.2 (D2)
- new net Keypad-4: MatrixMembraneKeypad1.3 (D3)
- new net Keypad-5: MatrixMembraneKeypad1.4 (D4)
- new net Keypad-6: MatrixMembraneKeypad1.5 (D5)
- new net Keypad-7: MatrixMembraneKeypad1.6 (D6)
- new net LCD-D4: LCD-1.11 (D4)
- new net LCD-D5: LCD-1.12 (D5)
- new net LCD-D6: LCD-1.13 (D6)
- new net LCD-D7: LCD-1.14 (D7)
- new net LCD-E: LCD-1.6 (E)
- new net LCD-RS: LCD-1.4 (RS)
- new net SrvM2-PWM-IN: SG1.1 (PWM)
- no-connect marks 3 -> 5
Other:
- title: Poubelle 1 -> Poubelle 2
